File: v1/Charakterograf.kicad_sch (KiCad schematic)
At the start: 85 parts, among them J2 X, J3 I_{C}=f(U_{CE}), J4 I_{C}=f(I_{BE}), J5 Y, P1 4k7, P2 47k, P3 10k, P4 47k, P5 47k, P6 10k, Q1 BC308, Q2 BC238, Q3 BD137, Q4 BD136, Q5 BD137, Q6 BD136, U1 LM555, U2 CD4520, U3 CD4051, U4 UA741, U5 UA741, U6 UA741, U7 UA741

Commit message: Fixed the mistake in one of the P/N switches
Parts:
- removed SW5: (no value), symbol custom:SW-SPDT-Flat_Basic
- added K3: (no value), symbol custom:Relay-Flat_Basic
Connections:
- net +15V: now also K3.
- net -15V: now also K3.
- net ±15V: now also K3.
- net at C5., R8.: now also SW2.; no longer U1.3
- net at U2.5 (D): now also U3.9 (C)
- new net: R26., R28., U6.2 (-)
- new net: R29., R30., SW7.
- new net: C7., J3. (E), Q3.1 (E), Q4.1 (E), R23., R37., R6., R7.
- new net: C4., P3., P4., P5.
- new net: C5., R8., U1.3
- new net: R13., R15., R16., R17., R18., R19., R20., R22., U4.3 (+), U4.6
- new net: R10., R11., SW4.
- new net: R35., R36., U3.7 (VEE)
- new net: R9., SW2., SW3.
- new net: R30., R31., SW7.
Changed lines of the file:
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@@
+	)
+	(symbol
+		(lib_id "custom:Relay-Flat_Basic")
+		(at 43.18 113.03 90)
+		(unit 2)
+		(body_style 1)
+		(exclude_from_sim no)
+		(in_bom yes)
+		(on_board yes)
+		(in_pos_files yes)
+		(dnp no)
+		(property "Reference" "K3"
+			(at 42.672 111.252 90)
+			(show_name no)
+			(do_not_autoplace no)
+			(effects
+				(font
+					(size 1.27 1.27)
+				)
+				(justify left)
+			)
+		)
+		(property "Value" ""
+			(at 43.18 113.03 0)
+			(show_name no)
+			(do_not_autoplace no)
+			(effects
+				(font
+					(size 1.27 1.27)
+				)
+			)
+		)
+		(property "Footprint" ""
+			(at 43.18 113.03 0)
+			(hide yes)
+			(show_name no)
+			(do_not_autoplace no)
+			(effects
+				(font
+					(size 1.27 1.27)
+				)
+			)
+		)
+		(property "Datasheet" ""
+			(at 43.18 113.03 0)
+			(hide yes)
+			(show_name no)
+			(do_not_autoplace no)
+			(effects
+				(font
+					(size 1.27 1.27)
+				)
+			)
+		)
+		(property "Description" ""
+			(at 43.18 113.03 0)
+			(hide yes)
+			(show_name no)
+			(do_not_autoplace no)
+			(effects
+				(font
+					(size 1.27 1.27)
+				)
+			)
+		)
+		(pin ""
+		)
+		(pin ""
+		)
+		(pin ""
+		)
+		(pin ""
+		)
+		(pin ""
+		)
+		(instances
+			(project "Charakterograf"
+				(path "/d7a5a570-e509-45ae-a7d3-ba88e6083368"
+					(reference "K3")
+					(unit 2)
+				)
+			)
+		)
 	)
 	(symbol
@@
 				)
 			)
-		)
-	)
-	(symbol
-		(lib_name "SW-SPDT-Flat_Basic_3")
-		(lib_id "custom:SW-SPDT-Flat_Basic")
-		(at 43.18 113.03 90)
-		(unit 1)
-		(body_style 1)
-		(exclude_from_sim no)
-		(in_bom yes)
-		(on_board yes)
-		(in_pos_files yes)
-		(dnp no)
-		(property "Reference" "SW5"
-			(at 42.672 110.998 90)
-			(show_name no)
-			(do_not_autoplace no)
-			(effects
-				(font
-					(size 1.27 1.27)
-				)
-				(justify left)
-			)
-		)
-		(property "Value" ""
-			(at 43.18 113.03 0)
-			(show_name no)
-			(do_not_autoplace no)
-			(effects
-				(font
-					(size 1.27 1.27)
-				)
-			)
-		)
-		(property "Footprint" ""
-			(at 43.18 113.03 0)
-			(hide yes)
-			(show_name no)
-			(do_not_autoplace no)
-			(effects
-				(font
-					(size 1.27 1.27)
-				)
-			)
-		)
-		(property "Datasheet" ""
-			(at 43.18 113.03 0)
-			(hide yes)
-			(show_name no)
-			(do_not_autoplace no)
-			(effects
-				(font
-					(size 1.27 1.27)
-				)
-			)
-		)
-		(property "Description" ""
-			(at 43.18 113.03 0)
-			(hide yes)
-			(show_name no)
-			(do_not_autoplace no)
-			(effects
-				(font
-					(size 1.27 1.27)
-				)
-			)
-		)
-		(pin ""
-		)
-		(pin ""
-		)
-		(pin ""
-		)
-		(instances
-			(project "Charakterograf"
-				(path "/d7a5a570-e509-45ae-a7d3-ba88e6083368"
-					(reference "SW5")
-					(unit 1)
-				)
-			)
