File: v2/untitled.kicad_sch (KiCad schematic)
At the start: 7 parts, among them P7 5k, U3 TL431, U4 OPA2277

Commit message: Added an unfinished pot stage
Connections:
- new net: C17., P7., R11., U3.4 (K), U4.6 (-)
