File: v2/5V_supply.kicad_sch (KiCad schematic)
At the start: 4 parts, among them U15 LM7805

Commit message: Almost finished v2
Parts:
- added D18: G LED, symbol Device:LED
- added R40: 1k, symbol custom:R_Basic
Connections:
- net 5V: now also R40.
- net GND: now also D18.1 (K)
- new net: D18.2 (A), R40.
