File: v2/Charakterograf.kicad_sch (KiCad schematic)
At the start: 67 parts, among them J2 X, J3 I_{C}=f(U_{CE}), J4 I_{C}=f(I_{BE}), J5 Y, P1 4k7, P2 47k, P3 10k, P4 47k, P5 47k, P6 10k, P7 5k, Q1 BC558C, Q2 BC548C, Q3 BD139, Q4 BD140, Q5 BD139, Q6 BD140, U1 NE555P, U10 TL072, U2 CD4520B, U3 TL431LP, U4 OPA2277, U5 TL072

Commit message: Increased page size, removed and started to improve for better the original switch
Parts:
- removed C17: 10u, symbol custom:C_Basic
- removed K1, K2: (no value), symbol custom:Basic_Relay
- removed K3: (no value), symbol custom:Relay-Flat_Basic
- removed K4: (no value), symbol custom:Relay_Basic
- removed P7: 5k, symbol custom:P-Trim_Basic
- removed R10, R11: 10k, symbol custom:R_Basic
- removed U3: TL431LP, Package_TO_SOT_THT:TO-92_Inline, symbol Reference_Voltage:TL431LP
- removed unit 2 of U4
- added C22, C23: 100n, symbol custom:C_Basic
- added J6: Sync, symbol Connector:Conn_Coaxial
- added J7: I_{C}=f(U_{CE}), symbol custom:3-Pin-Socket_Basic
- added K1, K2: (no value), symbol custom:Relay-Flat-DPDT_Basic
- added P8: Pot, symbol custom:P_Basic
- added R12: 1k, symbol custom:R_Basic
- added R4: R, symbol Device:R
- added SW4: (no value), symbol custom:SW-SP3T-Rotary_Basic
- added U11, U12, U7: ADG419BN, Package_DIP:DIP-8_W7.62mm, symbol Analog_Switch:ADG419BN
- added U6: TL071, DIP794W53P254L959H508Q8N, symbol custom:TL071
Connections:
- net +15V: now also C22., K2., U6.7 (+)
- net -15V: now also C23., K2., U6.4 (-)
- net GND: now also C22., C23., J6.2 (Ext), K1., K2.
- net ±15V: now also K2.
- net at R30., SW7.: now also R31.; no longer R29.
- net at C5., R8.: now also SW2.; no longer U1.3
- net at P6.: now also R5., U5.2 (-); no longer P5.
- net at J3. (E): now also J4. (E), R24., R25.
- net at U2.3 (A): now also U12.1
- net at U2.4 (B): now also U11.1
- net at U2.5 (D): now also U7.1
- new net: C4., K1.
- new net: K1., K1., P4., R33.
- new net: K1., K1., P5., P6.
- new net: R29., R30., SW7.
- new net: C7., J3. (E), Q3.3 (E), Q4.2 (C), R23., R37., R6., R7.
- new net: J7. (E), U6.3 (+), U6.6
- new net: C5., R12., R8., U1.3
- new net: J6.1 (In), R12.
- new net: R9., SW2., SW3.
- new net Vref: P8.
Other:
- sheet Swiches renamed N\P Swiches
- added sheet 8V Ref (ref.kicad_sch)
- added sheet Switch Supply (switch_supply.kicad_sch)
- note added: "Auto Step Pot"
- note removed: "0,1%"
- note removed: "Measure and trim so it's 8,000V"
- note removed: "Precision"

Commit message: Added an unfinished pot stage
Parts:
- removed P8: Pot, symbol custom:P_Basic
- removed R4: R, symbol Device:R
- added C30, C31, C9: 100n, symbol custom:C_Basic
- added P10: 10k, symbol custom:P_Basic
- added P9: 2k, symbol custom:P-Trim_Basic
- added R14: 10k, symbol custom:R_Basic
- added U13: OPA277, symbol custom:OPA277
Connections:
- net +15V: now also C30., U13.7 (+)
- net -15V: now also C31., U13.4 (-)
- net GND: now also C30., C31., P10.
- net Vref: now also P9.
- net at K1.: now also K1., P5., P6.; no longer C4.
- net at R30., SW7.: now also R31.; no longer R29.
- net at J7. (E): now also U6.3 (+), U6.6
- net at C5., R8.: now also SW2.; no longer R12., U1.3
- net at J3. (E): now also J4. (E), R24., R25.
- net at U2.5 (D): now also U7.1
- new net: C4., K1.
- new net: K1., K1., P4., R33.
- new net: R29., R30., SW7.
- new net: C9., P10., R14.
- new net: C9., R14., U13.2 (-)
- new net: C7., J3. (E), Q3.3 (E), Q4.2 (C), R23., R37., R6., R7.
- new net: C5., R12., R8., U1.3
- new net: P10., P9.
- new net: R9., SW2., SW3.
- new net: U13.3 (+), U13.6
Other:
- note removed: "Add clip-on heatsink"
- moved on the sheet: C1, C10, C11, C12, C13, C2, C22, C23, C3, C4, C5, C6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

Commit message: Almostt finished everything, just finishing details
Parts:
- removed C1, C12, C13, C2, C22, C23, C30, C31, C5, C6, C8, C9: 100n, symbol custom:C_Basic
- removed C10: 22n, symbol custom:C_Basic
- removed C11: 22u, symbol custom:C-Pol_Basic
- removed C3: 220n, symbol custom:C_Basic
- removed C4: 1u, symbol custom:C_Basic
- removed C7: 100p, symbol custom:C_Basic
- removed D10: 12V, symbol Device:D_Zener
- removed J2: X, symbol Connector:Conn_Coaxial
- removed J3, J7: I_{C}=f(U_{CE}), symbol custom:3-Pin-Socket_Basic
- removed J4: I_{C}=f(I_{BE}), symbol custom:3-Pin-Socket_Basic
- removed J5: Y, symbol Connector:Conn_Coaxial
- removed J6: Sync, symbol Connector:Conn_Coaxial
- removed K1, K2: (no value), symbol custom:Relay-Flat-DPDT_Basic
- removed P1: 4k7, symbol custom:P-Trim_Basic
- removed P10: 10k, symbol custom:P_Basic
- removed P2, P4, P5: 47k, symbol custom:P-Trim_Basic
- removed P3, P6: 10k, symbol custom:P-Trim_Basic
- removed P9: 2k, symbol custom:P-Trim_Basic
- removed Q1: BC558C, symbol Transistor_BJT:Q_PNP_CBE
- removed Q2: BC548C, symbol Transistor_BJT:Q_NPN_CBE
- removed Q3, Q5: BD139, symbol Transistor_BJT:Q_NPN_BCE
- removed Q4, Q6: BD140, symbol Transistor_BJT:Q_PNP_BCE
- removed R1: 4k7, symbol custom:R_Basic
- removed R12, R25, R27, R28, R34, R7: 1k, symbol custom:R_Basic
- removed R14, R2, R29, R30, R31, R33, R5, R8, R9: 10k, symbol custom:R_Basic
- removed R23: 20k, symbol custom:R_Basic
- removed R24: 1R, symbol custom:R_Basic
- removed R26: 100k, symbol custom:R_Basic
- removed R3: 47k, symbol custom:R_Basic
- removed R37, R38: 100R, symbol custom:R_Basic
- removed R6: 51k, symbol custom:R_Basic
- removed SW2, SW3, SW7: (no value), symbol custom:SW-SPDT-Flat_Basic
- removed SW4: (no value), symbol custom:SW-SP3T-Rotary_Basic
- removed U1: NE555P, Package_SO:SOIC-8_3.9x4.9mm_P1.27mm, symbol custom:LM555
- removed U10, U5: TL072, DIP794W53P254L959H508Q8N, symbol custom:TL072
- removed U11, U12, U7: ADG419BN, Package_DIP:DIP-8_W7.62mm, symbol Analog_Switch:ADG419BN
- removed U13: OPA277, symbol custom:OPA277
- removed U2: CD4520B, symbol custom:CD4520_basic
- removed U4: OPA2277, symbol Amplifier_Operational:OPA2277
- removed U6: TL071, DIP794W53P254L959H508Q8N, symbol custom:TL071
Connections:
- no-connect marks 1 -> 0
Other:
- sheet Power Supply renamed Power Supply Board
- removed sheet 8V Ref
- removed sheet N\P Swiches
- removed sheet Switch Supply
- added sheet Logic Board (Logic.kicad_sch)
- sheet Power Supply Board ports: added 12V; removed none
- note removed: "(I_{C}) 0,1V-1mA 1V-10mA 10V-100mA"
- note removed: "(U_{CE}) (I_{B}) 0-12V"
- note removed: "10V 5V"
- note removed: "A R"
- note removed: "Auto Step Pot"
- note removed: "I_{B}"
- note removed: "P N"

Commit message: Almost finished v2
Other:
- note added: "v3: -Add curren checker LM339 for relay coils -Add checking if all relays switched correcly -Add front pannel meter -Add step LEDs -Add external power option -Design HV Box"
Changed lines of the file:
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@@
 		(rev "2")
+	)
+	(text "v3:\n-Add curren checker LM339 for relay coils\n-Add checking if all relays switched correcly\n-Add front pannel meter\n-Add step LEDs\n-Add external power option\n-Design HV Box"
+		(exclude_from_sim no)
+		(at 13.97 29.718 0)
+		(effects
+			(font
+				(size 3 3)
+			)
+			(justify left)
+		)
 	)
 	(wire
 		(pts
-			(xy 154.94 58.42) (xy 151.13 58.42)
+			(xy 148.59 63.5) (xy 144.78 63.5)
 		)
 		(stroke
@@
 	(wire
 		(pts
-			(xy 151.13 54.61) (xy 154.94 54.61)
+			(xy 144.78 59.69) (xy 148.59 59.69)
 		)
 		(stroke
@@
 	(wire
 		(pts
-			(xy 151.13 62.23) (xy 154.94 62.23)
+			(xy 144.78 67.31) (xy 148.59 67.31)
 		)
 		(stroke
@@
 	(global_label "12V"
 		(shape output)
-		(at 154.94 62.23 0)
+		(at 148.59 67.31 0)
 		(fields_autoplaced yes)
 		(effects
@@
 		)
 		(property "Intersheetrefs" "${INTERSHEET_REFS}"
-			(at 161.4328 62.23 0)
+			(at 155.0828 67.31 0)
 			(hide yes)
 			(show_name no)
@@
 	(global_label "+15V"
 		(shape output)
-		(at 154.94 54.61 0)
+		(at 148.59 59.69 0)
 		(fields_autoplaced yes)
 		(effects
@@
 		)
 		(property "Intersheetrefs" "${INTERSHEET_REFS}"
-			(at 163.0052 54.61 0)
+			(at 156.6552 59.69 0)
 			(hide yes)
 			(show_name no)
@@
 	(global_label "-15V"
 		(shape output)
-		(at 154.94 58.42 0)
+		(at 148.59 63.5 0)
 		(fields_autoplaced yes)
 		(effects
@@
 		)
 		(property "Intersheetrefs" "${INTERSHEET_REFS}"
-			(at 163.0052 58.42 0)
+			(at 156.6552 63.5 0)
 			(hide yes)
 			(show_name no)
@@
 	)
 	(sheet
-		(at 124.46 49.53)
+		(at 118.11 54.61)
 		(size 26.67 19.05)
 		(exclude_from_sim no)
@@
 		)
 		(property "Sheetname" "Power Supply Board"
-			(at 124.46 48.8184 0)
+			(at 118.11 53.8984 0)
 			(show_name no)
 			(do_not_autoplace no)
@@
 		)
 		(property "Sheetfile" "power_supply.kicad_sch"
-			(at 124.46 69.1646 0)
+			(at 118.11 74.2446 0)
 			(hide yes)
 			(show_name no)
@@
 		)
 		(pin "+15V" output
-			(at 151.13 54.61 0)
+			(at 144.78 59.69 0)
 			(effects
 				(font
@@
 		)
 		(pin "-15V" output
-			(at 151.13 58.42 0)
+			(at 144.78 63.5 0)
 			(effects
 				(font
@@
 		)
 		(pin "12V" output
-			(at 151.13 62.23 0)
-			(effects
-				(font
+			(at 144.78 67.31 0)
+			(effects
+				(font
