File: v2/Unused.kicad_sch (KiCad schematic)
At the start: 2 parts, among them U13 CD40106B, U2 CD4520B

Commit message: Fixed incorrect wiring, wrong footprint, ec
Parts:
- removed U2: CD4520B, symbol custom:CD4520
- added U6: CD4520, symbol custom:CD4520
Connections:
- net 5V: now also U6.10 (EN), U6.15 (R), U6.9 (CL)
Changed lines of the file:
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@@
 		(instances
 			(project "Charakterograf"
-				(path "/d7a5a570-e509-45ae-a7d3-ba88e6083368/03491c05-b5f3-4f88-a242-4fe53ef90d21"
+				(path "/d7a5a570-e509-45ae-a7d3-ba88e6083368/03491c05-b5f3-4f88-a242-4fe53ef90d21/867728c2-15d3-4eb0-a7ff-a659d23fa9b9"
 					(reference "U13")
 					(unit 5)
-				)
-				(path "/d7a5a570-e509-45ae-a7d3-ba88e6083368/03491c05-b5f3-4f88-a242-4fe53ef90d21/867728c2-15d3-4eb0-a7ff-a659d23fa9b9"
-					(reference "U13")
-					(unit 5)
-				)
-			)
-		)
-	)
-	(symbol
-		(lib_name "CD4520_1")
-		(lib_id "custom:CD4520")
-		(at 149.86 73.66 0)
-		(unit 2)
-		(body_style 1)
-		(exclude_from_sim no)
-		(in_bom yes)
-		(on_board yes)
-		(in_pos_files yes)
-		(dnp no)
-		(fields_autoplaced yes)
-		(property "Reference" "U2"
-			(at 146.6215 58.42 0)
-			(show_name no)
-			(do_not_autoplace no)
-			(effects
-				(font
-					(size 1.27 1.27)
-				)
-			)
-		)
-		(property "Value" "CD4520B"
-			(at 146.6215 60.96 0)
-			(show_name no)
-			(do_not_autoplace no)
-			(effects
-				(font
-					(size 1.27 1.27)
-				)
-			)
-		)
-		(property "Footprint" ""
-			(at 149.86 73.66 0)
-			(hide yes)
-			(show_name no)
-			(do_not_autoplace no)
-			(effects
-				(font
-					(size 1.27 1.27)
-				)
-			)
-		)
-		(property "Datasheet" ""
-			(at 149.86 73.66 0)
-			(hide yes)
-			(show_name no)
-			(do_not_autoplace no)
-			(effects
-				(font
-					(size 1.27 1.27)
-				)
-			)
-		)
-		(property "Description" ""
-			(at 149.86 73.66 0)
-			(hide yes)
-			(show_name no)
-			(do_not_autoplace no)
-			(effects
-				(font
-					(size 1.27 1.27)
-				)
-			)
-		)
-		(pin "5"
-		)
-		(pin "12"
-		)
-		(pin "16"
-		)
-		(pin "4"
-		)
-		(pin "5"
-		)
-		(pin "7"
-		)
-		(pin "3"
-		)
-		(pin "15"
-		)
-		(pin "1"
-		)
-		(pin "13"
-		)
-		(pin "8"
-		)
-		(pin "10"
-		)
-		(pin "11"
-		)
-		(pin "2"
-		)
-		(pin "9"
-		)
-		(pin "14"
-		)
-		(instances
-			(project "Charakterograf"
-				(path "/d7a5a570-e509-45ae-a7d3-ba88e6083368/03491c05-b5f3-4f88-a242-4fe53ef90d21"
-					(reference "U2")
-					(unit 2)
-				)
-				(path "/d7a5a570-e509-45ae-a7d3-ba88e6083368/03491c05-b5f3-4f88-a242-4fe53ef90d21/867728c2-15d3-4eb0-a7ff-a659d23fa9b9"
-					(reference "U2")
-					(unit 2)
 				)
 			)
@@
 		(instances
 			(project "Charakterograf"
-				(path "/d7a5a570-e509-45ae-a7d3-ba88e6083368/03491c05-b5f3-4f88-a242-4fe53ef90d21"
+				(path "/d7a5a570-e509-45ae-a7d3-ba88e6083368/03491c05-b5f3-4f88-a242-4fe53ef90d21/867728c2-15d3-4eb0-a7ff-a659d23fa9b9"
 					(reference "U13")
 					(unit 4)
 				)
-				(path "/d7a5a570-e509-45ae-a7d3-ba88e6083368/03491c05-b5f3-4f88-a242-4fe53ef90d21/867728c2-15d3-4eb0-a7ff-a659d23fa9b9"
-					(reference "U13")
-					(unit 4)
+			)
+		)
+	)
+	(symbol
+		(lib_name "CD4520_2")
+		(lib_id "custom:CD4520")
+		(at 149.86 73.66 0)
+		(unit 2)
+		(body_style 1)
+		(exclude_from_sim no)
+		(in_bom yes)
+		(on_board yes)
+		(in_pos_files yes)
+		(dnp no)
+		(fields_autoplaced yes)
+		(property "Reference" "U6"
+			(at 146.6215 58.42 0)
+			(show_name no)
+			(do_not_autoplace no)
+			(effects
+				(font
+					(size 1.27 1.27)
+				)
+			)
+		)
+		(property "Value" "CD4520"
+			(at 146.6215 60.96 0)
+			(show_name no)
+			(do_not_autoplace no)
+			(effects
+				(font
+					(size 1.27 1.27)
+				)
+			)
+		)
+		(property "Footprint" ""
+			(at 149.86 73.66 0)
+			(hide yes)
+			(show_name no)
+			(do_not_autoplace no)
+			(effects
+				(font
+					(size 1.27 1.27)
+				)
+			)
+		)
+		(property "Datasheet" ""
+			(at 149.86 73.66 0)
+			(hide yes)
+			(show_name no)
+			(do_not_autoplace no)
+			(effects
+				(font
+					(size 1.27 1.27)
+				)
+			)
+		)
+		(property "Description" ""
+			(at 149.86 73.66 0)
+			(hide yes)
+			(show_name no)
+			(do_not_autoplace no)
+			(effects
+				(font
+					(size 1.27 1.27)
+				)
+			)
+		)
+		(pin "12"
+		)
+		(pin "8"
+		)
+		(pin "9"
+		)
+		(pin "5"
+		)
+		(pin "10"
+		)
+		(pin "13"
+		)
+		(pin "14"
+		)
+		(pin "3"
+		)
+		(pin "7"
+		)
+		(pin "16"
+		)
+		(pin "1"
+		)
+		(pin "2"
+		)
+		(pin "6"
+		)
+		(pin "4"
+		)
+		(pin "11"
+		)
+		(pin "15"
+		)
+		(instances
+			(project "Charakterograf"
+				(path "/d7a5a570-e509-45ae-a7d3-ba88e6083368/03491c05-b5f3-4f88-a242-4fe53ef90d21"
+					(reference "U6")
+					(unit 2)
+				)
+				(path "/d7a5a570-e509-45ae-a7d3-ba88e6083368/03491c05-b5f3-4f88-a242-4fe53ef90d21/867728c2-15d3-4eb0-a7ff-a659d23fa9b9"
+					(reference "U6")
+					(unit 2)
 				)
 			)
@@
 		(instances
 			(project "Charakterograf"
-				(path "/d7a5a570-e509-45ae-a7d3-ba88e6083368/03491c05-b5f3-4f88-a242-4fe53ef90d21"
-					(reference "U13")
-					(unit 3)
-				)
 				(path "/d7a5a570-e509-45ae-a7d3-ba88e6083368/03491c05-b5f3-4f88-a242-4fe53ef90d21/867728c2-15d3-4eb0-a7ff-a659d23fa9b9"
 					(reference "U13")
@@
 		(instances
 			(project "Charakterograf"
-				(path "/d7a5a570-e509-45ae-a7d3-ba88e6083368/03491c05-b5f3-4f88-a242-4fe53ef90d21"
-					(reference "U13")
-					(unit 2)
-				)
 				(path "/d7a5a570-e509-45ae-a7d3-ba88e6083368/03491c05-b5f3-4f88-a242-4fe53ef90d21/867728c2-15d3-4eb0-a7ff-a659d23fa9b9"
 					(reference "U13")
@@
 		(instances
 			(project "Charakterograf"
-				(path "/d7a5a570-e509-45ae-a7d3-ba88e6083368/03491c05-b5f3-4f88-a242-4fe53ef90d21"
+				(path "/d7a5a570-e509-45ae-a7d3-ba88e6083368/03491c05-b5f3-4f88-a242-4fe53ef90d21/867728c2-15d3-4eb0-a7ff-a659d23fa9b9"
 					(reference "U13")
-					(unit 6)
-				)
-				(path "/d7a5a570-e509-45ae-a7d3-ba88e6083368/03491c05-b5f3-4f88-a242-4fe53ef90d21/867728c2-15d3-4eb0-a7ff-a659d23fa9b9"
-					(reference "U13")
