File: v2/Logic.kicad_sch (KiCad schematic)
At the start: 89 parts, among them J2 X, J5 Y, J6 Sync, J7 I_{C}=f(U_{CE}), P1 4k7, P10 10k, P2 47k, P3 10k, P4 47k, P5 47k, P6 10k, P9 2k, Q1 BC558C, Q2 BC548C, Q3 BD139, Q4 BD140, Q5 BD139, Q6 BD140, U1 NE555P, U10 TL072, U11 ADG419BN, U12 ADG419BN, U16 OPA2277, U17 OPA2277, U2 CD4520B, U4 OPA2277, U5 TL072, U6 TL071, U7 ADG419BN

Commit message: Almost finished v2
Parts:
- removed C9: 100n, symbol custom:C_Basic
- removed SW2, SW3: (no value), symbol custom:SW-SPDT-Flat_Basic
- removed U2: CD4520B, symbol custom:CD4520_basic
- added C11: 470n, symbol custom:C_Basic
- added C43, C45: 100n, symbol custom:C_Basic
- added C44: 47p, symbol custom:C_Basic
- added P11, P8: 200R, symbol custom:P-Trim_Basic
- added P12: 20k, symbol custom:P-Trim_Basic
- added R21, R22: 10k, symbol custom:R_Basic
- added R42, R43, R47, R48, R49, R50, R51, R52, R53, R54: 100k, symbol custom:R_Basic
- added R45, R46: 20k, symbol custom:R_Basic
- added SW10: (no value), symbol custom:SW-SP3T_Basic
- added SW2: I_{B}, symbol Switch:SW_Push
- added SW3: (no value), symbol custom:SW-DP4T-Rotary_Basic
- added U13: CD40106B, symbol custom:CD40106B
- added U2: CD4520B, symbol custom:CD4520
- R26: value 100k -> 91k
- renumbered C5 to C9, R23 to R44
Connections:
- net 12V is gone; now on net 5V: R9.
- net 5V: now also C43., U13.14 (+), U2.16 (+), U2.2 (EN)
- net GND: now also D1.2 (A), D2.1 (K), K2., C11., C43., C45., R47., R49., R51., R53., SW2.2, U13.7 (-), U2.7 (R), U2.8 (GND)
- net at Q5.3 (E), Q6.3 (E), R38.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: now also SW6.2 (B)
- net at K1.: now also K1., P5., P6.; no longer C4.
- net at R29.: now also R30., SW7.; no longer K2.
- net at R30., SW7.: now also R31.; no longer R29.
- net at R14.: now also U16.3 (+), C45.; no longer P10.
- net at SW8.1 (A), SW8.1 (A), SW8.1 (A): now also SW9.2 (B); no longer J7. (E)
- net at U11.6: now also U2.4 (B)
- net at C9., R8.: now also SW4.1 (A); no longer R12., U1.3
- net at D1.1 (K), D2.2 (A): now also R25., U4.3 (+)
- net at SW4.2 (B): now also U2.1 (CL)
- net at SW4.3 (C): now also SW4.1 (A), U13.2
- net at R44., SW6.1 (A), SW8.2 (B)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: now also R45., R46.
- net at R44.: now also SW10.4; no longer SW6.3 (C)
- net at U12.6: now also U2.3 (A)
- net at SW6.2 (B): now also C7., Q3.3 (E), Q4.2 (C), R37., R6., R7., SW5.1 (A)
- net at U17.5 (+): now also R48., R50., R52., R54., SW3.2 (B)
- net at U17.6 (-): now also SW6.2 (B), C44., P11., R42.
- net at U17.7: now also C44., R43., SW3.2 (B)
- net at U7.6: now also U2.5 (D)
- net at R25.: now also R24., SW8.2 (B); no longer U4.3 (+)
- net at U17.1: now also R22., R42.
- net at U17.2 (-): now also P8., R21.
- net at SW4.2 (B): now also K2., R21.
- new net: R16., R19., R20.
- new net: R15., R18., R20.
- new net: C4., K1.
- new net: K1., K1., P4., R33.
- new net: K2., R29.
- new net: C11., R9., SW2.1, U13.1
- new net: C1., C5., Q2.1 (C), R1., R2., R4., U1.4, U1.8
- new net: J7. (E), SW8.1 (A), SW8.1 (A), SW8.1 (A)
- new net: C9., R12., R8., U1.3
- new net: P10., P9.
- new net: P10., R14.
- new net: R49., SW3.1 (A)
- new net: R52., SW3.1 (A)
- new net: R54., SW3.1 (A)
- new net: R50., SW3.1 (A)
- new net: SW8.1 (A), SW8.1 (A), SW8.1 (A), SW9.2 (B)
- new net: SW10.3, SW6.3 (C)
- new net: R48., SW3.3 (C)
- new net: P11., R43.
- new net: R46., SW10.1
- new net: R45., SW10.2
- new net: P12., R26.
- new net: R51., SW3.1 (A)
- new net: P12., R28., U4.2 (-)
- new net: P8., R22.
- new net: R53., SW3.1 (A)
- new net: R47., SW3.3 (C)
- no-connect marks 1 -> 6
Other:
- added sheet Unused Parts (Unused.kicad_sch)
- note added: "(V_{CE}) (I_{B}) 0-12V"
- note added: "C/E Inverter"
- note added: "Make it locking"
- note added: "Matched 0,1%"
- note added: "Pinout"
- note added: "R44-20k R45-47k R46-100k"
- note added: "R47/48-1M R49/50-100k R51/52-10k R53/54-1k"
- note added: "Set to 99k"
- note added: "V_{CE}/I_{BE}"
- note removed: "(U_{CE}) (I_{B}) 0-12V"
- note removed: "/C"
- note removed: "A R"
- note removed: "B/"
- note removed: "C/B"
- note removed: "Either matched or 0,1%"
- note removed: "I_{B}"
- moved on the sheet: C1, C10, C12, C13, C2, C22, C23, C3, C30, C31, C4, C41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

Commit message: Fixed incorrect wiring, wrong footprint, ec
Parts:
- removed C22, C23: 100n, symbol custom:C_Basic
- removed U2: CD4520B, symbol custom:CD4520
- removed U6: TL071, DIP794W53P254L959H508Q8N, symbol custom:TL071
- added R23: 100k, symbol custom:R_Basic
- added R56: 10R, symbol custom:R_Basic
- added R57: 1R, symbol custom:R_Basic
- added SW12: (no value), symbol custom:SW-DP3T_Basic
- added U6: CD4520, symbol custom:CD4520
- R45: value 20k -> 47k
- R46: value 20k -> 100k
- R47, R48: value 100k -> 1M
- R51, R52: value 100k -> 10k
- R53, R54: value 100k -> 1k
- R55: renamed from R24; value 1R -> 100R
- renumbered U10 to U5
Connections:
- net -15V: now also Q4.2 (C); no longer Q4.3 (E)
- net 5V: now also U6.16 (+), U6.2 (EN)
- net GND: now also SW8.3 (C), R23., R56., R57., U6.7 (R), U6.8 (GND)
- net at K1.: now also K1., P5., P6.; no longer C4.
- net at R29.: now also R30., SW7.; no longer K2.
- net at R30., SW7.: now also R31.; no longer R29.
- net at C7., R33., R6.: now also U5.2 (-); no longer U5.3 (+)
- net at SW9.1 (A), SW9.3 (C): now also SW8.2 (B); no longer J7. (E) (x2)
- net at U11.6: now also U6.4 (B)
- net at K2., R21., SW4.2 (B): now also R23.
- net at SW6.1 (A), SW6.3 (C): now also SW9.2 (B); no longer SW8.2 (B)
- net at C9., R8.: now also SW4.1 (A); no longer R12., U1.3
- net at R14.: now also C45., U16.3 (+); no longer P10.
- net at SW3.1 (A): now also R53.; no longer R49.
- net at SW4.2 (B): now also U6.1 (CL)
- net at U12.6: now also U6.3 (A)
- net at U7.6: now also U6.5 (C)
- new net: R16., R19., R20.
- new net: R15., R18., R20.
- new net: C4., K1.
- new net: K1., K1., P4., R33.
- new net: K2., R29.
- new net: C44., P11., R42., SW6.2 (B), U17.6 (-)
- new net: C7., Q3.3 (E), Q4.3 (E), R37., R6., R7., SW5.1 (A), SW6.2 (B)
- new net: C1., C5., Q2.1 (C), R1., R2., R4., U1.4, U1.8
- new net: J7. (E), SW8.1 (A), SW8.1 (A), SW8.1 (A) (x2)
- new net: P8., R21., U17.2 (-)
- new net: R55., SW12.1, SW12.1
- new net: R56., SW12.2, SW12.2
- new net: R25., SW12.3
- new net: R57., SW12.4, SW12.4
- new net: C9., R12., R8., U1.3
- new net: P10., P9.
- new net: P10., R14.
- new net: R49., SW3.1 (A)
- new net: R48., R50., R52., R54., SW3.2 (B), U17.5 (+)
- new net: R44., R45., R46., SW6.1 (A), SW8.2 (B)
- new net: R51., SW3.1 (A)
- new net: P6., R5., U5.3 (+)
- new net: SW12.3, SW9.2 (B)
- no-connect marks 6 -> 5
Other:
- note added: "All switches are break-before-make except for 2"
- note added: "Make-before-break"
- note added: "R55 100R 0,1% R56 10R 0,1% R57 1R 0,1% ^{1}/_{2}W"
- note removed: "Non-shorting"
- note removed: "To meter for base"
- moved on the sheet: C12, C13, D1, D2, J5, P12, R25, R26, R27, R28, R55, SW8A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

Commit message: Finished, adding minure debug and production stuff, need to make PCB
Parts:
- added R59: 47R, symbol custom:R_Basic
- added R60: 470R, symbol custom:R_Basic
- added R61: 4k7, symbol custom:R_Basic
- added SW11: (no value), symbol custom:SW-SP4T_Basic
- J7: value I_{C}=f(U_{CE}) -> (none)
- R22: value 10k -> 9k88
- R43: value 100k -> 99k8
Connections:
- net at K1.: now also K1., P5., P6.; no longer C4.
- net at R29.: now also R30., SW7.; no longer K2.
- net at R30., SW7.: now also R31.; no longer R29.
- net at SW6.3 (C), SW9.2 (B): now also R59., R60., R61., SW11.4; no longer SW6.1 (A)
- net at C9., R8.: now also SW4.1 (A); no longer R12., U1.3
- net at R14.: now also C45., U16.3 (+); no longer P10.
- net at SW3.1 (A): now also R53.; no longer R49.
- new net: R16., R19., R20.
- new net: R15., R18., R20.
- new net: C4., K1.
- new net: K1., K1., P4., R33.
- new net: K2., R29.
- new net: C44., P11., R42., U17.6 (-)
- new net: C1., C5., Q2.1 (C), R1., R2., R4., U1.4, U1.8
- new net: J7. (E), SW8.1 (A), SW8.1 (A), SW8.1 (A) (x2)
- new net: P8., R21., U17.2 (-)
- new net: R60., SW11.2
- new net: C9., R12., R8., U1.3
- new net: P10., P9.
- new net: P10., R14.
- new net: R49., SW3.1 (A)
- new net: R48., R50., R52., R54., SW3.2 (B), SW6.2 (B), U17.5 (+)
- new net: R44., R45., R46., SW6.1 (A), SW8.2 (B)
- new net: SW11.3, SW6.1 (A)
- new net: R59., SW11.1
- new net: R51., SW3.1 (A)
- new net: R61., SW11.4
Other:
- note added: "R59 47R 2W R60 470R ^{1}/_{2}W R61 4k7"
- note removed: "All switches are break-before-make except for 2"
- note removed: "Make it locking"
- note removed: "Make-before-break"
- note removed: "Set to 99k"
- moved on the sheet: C44, P11, P8, R22, R42, R43, R47, R48, R49, R50, R51, R52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
