File: v2/power_supply.kicad_sch (KiCad schematic)
At the start: 16 parts, among them J1 Screw_Terminal_01x03, U8 L7815, U9 L7915

Commit message: Increased page size, removed and started to improve for better the original switch
Connections:
- new net: C16., C19.
Changed lines of the file:
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@@
 		(title "Curve Plotter")
 		(date "2026-10-15")
-		(rev "1")
+		(rev "2")
 	)
 	(text "Use a standart IEC C14 socket with a built in fuse holder\nUse a slow-blow (T) 250V AC fuse (160mA for 15VA or 250mA for 30VA)"

Commit message: Almostt finished everything, just finishing details
Parts:
- added C35, C36: 100n, symbol custom:C_Basic
- added C37: 47u, symbol custom:C-Pol_Basic
- added D17: G LED, symbol Device:LED
- added R34: 2k, symbol custom:R_Basic
- added U14: LM7812, Package_TO_SOT_THT:TO-220-3_Vertical, symbol Regulator_Linear:LM7812_TO220
- U8: value L7815 -> LM7815
- U9: value L7915 -> LM7915
Connections:
- net GND: now also C35., C36., C37., D17.1 (K), U14.2 (GND)
- net at C18., C20., D6.4 (+)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: now also C35., U14.1 (VI)
- new net: D17.2 (A), R34.
- new net: C16., C19.
- new net 12V: C36., C37., R34., U14.3 (VO)
Other:
- moved on the sheet: C14, C15, C16, C18, C19, C20, C21, D15, D16, D6, J1, R32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

Commit message: Almost finished v2
Parts:
- added D10, D11, D12: 1N4007, Diode_THT:D_DO-35_SOD27_P7.62mm_Horizontal, symbol Diode:1N4148
- added D3, D4: 1N5819, symbol Device:D_Schottky
- added F1, F2, F3: A5 hold 30V, symbol custom:F-poly_Basic
- C20, C21: value 470u -> 2200u
- R34: value 2k -> 3k3
- renumbered C19 to C17
Connections:
- net +15V: now also D10.2 (A), D3.1 (K), F1.
- net -15V: now also D11.1 (K), D4.2 (A), F2.
- net 12V: now also D12.2 (A), F3.
- net GND: now also D3.2 (A), D4.1 (K), F1., F2., F3.
- net at C18., C20., C35.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: now also D10.1 (K), D12.1 (K)
- net at C19., C21., D6.1 (-)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: now also D11.2 (A)
- new net: C16., C17.
Other:
- note added: "KBP206 or 4x1N5408"
- note removed: "Build In Full Bridge Rectifier or 4x1N5401-1N5408"
- moved on the sheet: C14, C15, C16, C17, C18, C19, C20, C21, C35, C36, C37, D15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

Commit message: Fixed incorrect wiring, wrong footprint, ec
Parts:
- D6: value B40C2300-1500A -> KBP206
Connections:
- net +15V: no longer C14., C16., D10.2 (A), D3.1 (K), R32., U8.3 (OUT)
- net -15V: no longer C15., C17., D11.1 (K), D4.2 (A), R35., U9.3 (VO)
- net 12V: no longer C36., C37., D12.2 (A), R34., U14.3 (VO)
- net GND: no longer F1., F2., F3.
- new net: C14., C16., D10.2 (A), D3.1 (K), F1., R32., U8.3 (OUT)
- new net: C15., C17., D11.1 (K), D4.2 (A), F2., R35., U9.3 (VO)
- new net: C36., C37., D12.2 (A), F3., R34., U14.3 (VO)
Other:
- moved on the sheet: F1, F2, F3

Commit message: Finished, adding minure debug and production stuff, need to make PCB
Parts:
- removed D6: KBP206, Diode_THT:Diode_Bridge_19.0x3.5x10.0mm_P5.0mm, symbol Diode_Bridge:B40C2300-1500A
- added D19, D20, D5, D6: 1N5408, Diode_THT:D_DO-201AD_P15.24mm_Horizontal, symbol Diode:1N5408
Connections:
- net +15V: now also R32.
- net -15V: now also R35.
- net 12V: now also R34.
- net at C18., C20., C35.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: now also D5.1 (K), D6.1 (K)
- net at C19., C21., D11.2 (A)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: now also D19.2 (A), D20.2 (A)
- net at J1.1 (Pin_1): now also D20.1 (K), D6.2 (A)
- net at J1.3 (Pin_3): now also D19.1 (K), D5.2 (A)
- new net: C14., C16., D10.2 (A), D3.1 (K), F1., U8.3 (OUT)
- new net: C15., C17., D11.1 (K), D4.2 (A), F2., U9.3 (VO)
- new net: C36., C37., D12.2 (A), F3., U14.3 (VO)
Other:
- note removed: "KBP206 or 4x1N5408"
- moved on the sheet: C14, C15, C16, C17, C18, C19, C20, C21, C35, C36, C37, D10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
