File: v2/swiches.kicad_sch (KiCad schematic)
At the start: 17 parts, among them Q7 BD139

Commit message: Increased page size, removed and started to improve for better the original switch
Parts:
- removed D10, D8: 1N4148, Diode_THT:D_DO-35_SOD27_P7.62mm_Horizontal, symbol Diode:1N4148
- removed K1, K2: (no value), symbol custom:Basic_Relay
- removed K3, K4: (no value), symbol custom:Relay_Basic
- removed Q7: BD139, symbol Transistor_BJT:Q_NPN_BCE
- added K1, K2: (no value), symbol custom:Relay-Flat-DPDT_Basic
- added Q7: BC548C, symbol Transistor_BJT:Q_NPN_CBE
Connections:
- net +15V: now also K1., K2.
- net GND: now also Q7.3 (E)
- net at D12.2 (A), D7.2 (A), D9.2 (A)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: now also K1., K2.
- net at R41.: now also Q7.2 (B)
- new net: Q7.1 (C), R40.
Other:
- note added: "For any number of relays: R_{40} = ^{V}/_{IC} - (^{1}/_{Rc1} + ^{1}/_{Rc2} + ...)^{-1} Ic = ^{Vc}/_{Rc} IC = Ic1 + Ic2 + ... I = ^{V}/_{R} R = R_{40} + (^{1}/_{Rc1} + ^{1}/_{Rc2} + ...)^{-1} R_{41} = ^{V}/_{Ib} Ib = ^{I}/_{10} W_{R40} = R_{40} * I^{2} W_{R41} = R_{41} * Ib^{2}"
- note added: "V-Supply Voltage Vc-Coil Voltage I-Supply Curren Ic-Coil Current IC-Total Coil Current Ib-Base Current R-Colector Reistance Rc-Coil Resistance R_{40}-R40 Resistance R_{41}-R41 Resistance W_{R40}-R_{40} Power W_{R41}-R_{41} Power nK-Number of Relays"
- note added: "check max switch currentt rating if too much use transistor"
- note added: "replace for a smaller voltage"
- note removed: "For any number of relays: R_{40} = ^{V}/_{Ic*nK} - ^{Rc}/_{nK} Ic = ^{Vc}/_{Rc} I = ^{V}/_{R} R = R_{40} + ^{Rc}/_{nK} R_{41} = ^{V}/_{Ib} Ib = ^{I}/_{10} W_{R40} = R_{40} * I^{2} W_{R41} = R_{41} * Ib^{2}"
- note removed: "V-Supply Voltage Vc-Coil Voltage I-Supply Curren Ic-Coil Current Ib-Base Current R-Colector Reistance Rc-Coil Resistance R_{40}-R40 Resistance R_{41}-R41 Resistance W_{R40}-R_{40} Power W_{R41}-R_{41} Power nK-Number of Relays"
- moved on the sheet: D12, D13, D14, D9, K6A, K6B, R39

Commit message: Almostt finished everything, just finishing details
Parts:
- removed R40: 47R, symbol custom:R_Basic
- Q7: value BC548C -> BC337
- R39: value 680R -> 560R
Connections:
- net at Q7.1 (C): now also D12.2 (A), D7.2 (A), D9.2 (A), K1., K2., K6.
- net 12V: now reaches K1., K2., K6.
- net 12V: now also D12.1 (K), D7.1 (K), D9.1 (K), K6.; no longer D12.2 (A), D7.2 (A), D9.2 (A)
- removed net +15V: D12.1 (K), D7.1 (K), D9.1 (K), K1., K2., K6., K6., SW1.2 (B)
- new net 5V: SW1.2 (B)
Other:
- note added: "Calculate R41"
- note added: "For any number of relays: I = ^{Vc}/_{R} I = Ic1 + Ic2 + ... R = (^{1}/_{Rc1} + ^{1}/_{Rc2} + ...)^{-1} R_{41} = ^{Vs}/_{Ib} Ib = ^{Ic}/_{10} W_{R41} = R_{41} * Ib^{2}"
- note added: "If I ≥ 800mA replace transistor"
- note added: "Vc-Coil Voltage Vs-Switch Voltage I-Collector Curren Ic-Coil Current Ib-Base Current R-Collector Resistance Rc-Coil Resistance R_{41}-R41 Resistance W_{R41}-R_{41} Power"
- note removed: "For any number of relays: R_{40} = ^{V}/_{IC} - (^{1}/_{Rc1} + ^{1}/_{Rc2} + ...)^{-1} Ic = ^{Vc}/_{Rc} IC = Ic1 + Ic2 + ... I = ^{V}/_{R} R = R_{40} + (^{1}/_{Rc1} + ^{1}/_{Rc2} + ...)^{-1} R_{41} = ^{V}/_{Ib} Ib = ^{I}/_{10} W_{R40} = R_{40} * I^{2} W_{R41} = R_{41} * Ib^{2}"
- note removed: "Might need to be ^{1}/_{2}W"
- note removed: "V-Supply Voltage Vc-Coil Voltage I-Supply Curren Ic-Coil Current IC-Total Coil Current Ib-Base Current R-Colector Reistance Rc-Coil Resistance R_{40}-R40 Resistance R_{41}-R41 Resistance W_{R40}-R_{40} Power W_{R41}-R_{41} Power nK-Number of Relays"
- note removed: "check max switch currentt rating if too much use transistor"
- note removed: "replace for a smaller voltage"
- moved on the sheet: D12, D13, D14, D7, D9, K1A, K2A, K6A, K6B, R39

Commit message: Almost finished v2
Parts:
- renumbered D9 to D8, D12 to D9
Other:
- note added: "D7 - D9 1N4148"
- note removed: "D7 - D12 1N4148"
Changed lines of the file:
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@@
 		)
 	)
-	(text "D7 - D12 1N4148"
+	(text "D7 - D9 1N4148"
 		(exclude_from_sim no)
 		(at 94.742 100.584 0)
@@
 		(in_pos_files yes)
 		(dnp no)
-		(property "Reference" "D9"
+		(property "Reference" "D8"
 			(at 117.602 107.95 90)
 			(show_name no)
@@
 			(project "Charakterograf"
 				(path "/d7a5a570-e509-45ae-a7d3-ba88e6083368/03491c05-b5f3-4f88-a242-4fe53ef90d21/007af530-feb9-4f03-aaed-db03e570bb53"
-					(reference "D9")
+					(reference "D8")
 					(unit 1)
 				)
@@
 		(in_pos_files yes)
 		(dnp no)
-		(property "Reference" "D12"
+		(property "Reference" "D9"
 			(at 134.366 107.95 90)
 			(show_name no)
@@
 			(project "Charakterograf"
 				(path "/d7a5a570-e509-45ae-a7d3-ba88e6083368/03491c05-b5f3-4f88-a242-4fe53ef90d21/007af530-feb9-4f03-aaed-db03e570bb53"
-					(reference "D12")
+					(reference "D9")
 					(unit 1)
 				)

Commit message: Fixed incorrect wiring, wrong footprint, ec
Parts:
- added R58: 10k, symbol custom:R_Basic
- R39: value 560R -> 2k2
Connections:
- net GND: now also R58.
- net at Q7.2 (B), R41.: now also R58.
Other:
- moved on the sheet: R41, SW1
Changed lines of the file:
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@@
 		(color 0 0 0 0)
 	)
+	(junction
+		(at 99.06 124.46)
+		(diameter 0)
+		(color 0 0 0 0)
+	)
 	(wire
 		(pts
@@
 	(wire
 		(pts
-			(xy 74.93 124.46) (xy 77.47 124.46)
+			(xy 73.66 124.46) (xy 76.2 124.46)
 		)
 		(stroke
@@
 	(wire
 		(pts
+			(xy 99.06 124.46) (xy 99.06 125.73)
+		)
+		(stroke
+			(width 0)
+			(type default)
+		)
+	)
+	(wire
+		(pts
 			(xy 154.94 100.33) (xy 154.94 102.87)
 		)
@@
 	(wire
 		(pts
-			(xy 87.63 124.46) (xy 88.9 124.46)
+			(xy 99.06 135.89) (xy 99.06 137.16)
+		)
+		(stroke
+			(width 0)
+			(type default)
+		)
+	)
+	(wire
+		(pts
+			(xy 86.36 124.46) (xy 87.63 124.46)
 		)
 		(stroke
@@
 	(wire
 		(pts
+			(xy 99.06 124.46) (xy 100.33 124.46)
+		)
+		(stroke
+			(width 0)
+			(type default)
+		)
+	)
+	(wire
+		(pts
 			(xy 152.4 121.92) (xy 152.4 120.65)
 		)
@@
 	(wire
 		(pts
-			(xy 99.06 124.46) (xy 100.33 124.46)
+			(xy 97.79 124.46) (xy 99.06 124.46)
 		)
 		(stroke
@@
 	(global_label "5V"
 		(shape input)
-		(at 74.93 124.46 180)
+		(at 73.66 124.46 180)
 		(fields_autoplaced yes)
 		(effects
@@
 		)
 		(property "Intersheetrefs" "${INTERSHEET_REFS}"
-			(at 69.6467 124.46 0)
+			(at 68.3767 124.46 0)
 			(hide yes)
 			(show_name no)
@@
 	(symbol
 		(lib_id "custom:SW-SPST_Basic")
-		(at 82.55 124.46 0)
+		(at 81.28 124.46 0)
 		(unit 1)
 		(body_style 1)
@@
 		(fields_autoplaced yes)
 		(property "Reference" "SW1"
-			(at 82.55 119.38 0)
+			(at 81.28 119.38 0)
 			(show_name no)
 			(do_not_autoplace no)
@@
 		)
 		(property "Value" ""
-			(at 82.55 124.46 0)
+			(at 81.28 124.46 0)
 			(show_name no)
 			(do_not_autoplace no)
@@
 		)
 		(property "Footprint" ""
-			(at 82.55 124.46 0)
+			(at 81.28 124.46 0)
 			(hide yes)
 			(show_name no)
@@
 		)
 		(property "Datasheet" ""
-			(at 82.55 124.46 0)
+			(at 81.28 124.46 0)
 			(hide yes)
 			(show_name no)
@@
 		)
 		(property "Description" ""
-			(at 82.55 124.46 0)
+			(at 81.28 124.46 0)
 			(hide yes)
 			(show_name no)
@@
 			)
 		)
-		(property "Value" "560R"
+		(property "Value" "2k2"
 			(at 160.02 129.5399 90)
 			(show_name no)
@@
 				(path "/d7a5a570-e509-45ae-a7d3-ba88e6083368/03491c05-b5f3-4f88-a242-4fe53ef90d21/007af530-feb9-4f03-aaed-db03e570bb53"
 					(reference "D7")
+					(unit 1)
+				)
+			)
+		)
+	)
+	(symbol
+		(lib_name "R_Basic_1")
+		(lib_id "custom:R_Basic")
+		(at 99.06 130.81 270)
+		(unit 1)
+		(body_style 1)
+		(exclude_from_sim no)
+		(in_bom yes)
+		(on_board yes)
+		(in_pos_files yes)
+		(dnp no)
+		(fields_autoplaced yes)
+		(property "Reference" "R58"
+			(at 101.6 129.5399 90)
+			(show_name no)
+			(do_not_autoplace no)
+			(effects
+				(font
+					(size 1.27 1.27)
+				)
+				(justify left)
+			)
+		)
+		(property "Value" "10k"
+			(at 101.6 132.0799 90)
+			(show_name no)
+			(do_not_autoplace no)
+			(effects
+				(font
+					(size 1.27 1.27)
+				)
+				(justify left)
+			)
+		)
+		(property "Footprint" ""
+			(at 99.06 130.81 0)
+			(hide yes)
+			(show_name no)
+			(do_not_autoplace no)
+			(effects
+				(font
+					(size 1.27 1.27)
+				)
+			)
+		)
+		(property "Datasheet" ""
+			(at 99.06 130.81 0)
+			(hide yes)
+			(show_name no)
+			(do_not_autoplace no)
+			(effects
+				(font
+					(size 1.27 1.27)
+				)
+			)
+		)
+		(property "Description" ""
+			(at 99.06 130.81 0)
+			(hide yes)
+			(show_name no)
+			(do_not_autoplace no)
+			(effects
+				(font
+					(size 1.27 1.27)
+				)
+			)
+		)
+		(pin ""
+		)
+		(pin ""
+		)
+		(instances
+			(project "Charakterograf"
+				(path "/d7a5a570-e509-45ae-a7d3-ba88e6083368/03491c05-b5f3-4f88-a242-4fe53ef90d21/007af530-feb9-4f03-aaed-db03e570bb53"
+					(reference "R58")
 					(unit 1)
 				)
@@
 	)
 	(symbol
+		(lib_id "power:GND")
+		(at 99.06 137.16 0)
+		(unit 1)
+		(body_style 1)
+		(exclude_from_sim no)
+		(in_bom yes)
+		(on_board yes)
+		(in_pos_files yes)
+		(dnp no)
+		(fields_autoplaced yes)
+		(property "Reference" "#PWR016"
+			(at 99.06 143.51 0)
+			(hide yes)
+			(show_name no)
+			(do_not_autoplace no)
+			(effects
+				(font
+					(size 1.27 1.27)
+				)
+			)
+		)
+		(property "Value" "GND"
+			(at 99.06 142.24 0)
+			(hide yes)
+			(show_name no)
+			(do_not_autoplace no)
+			(effects
+				(font
+					(size 1.27 1.27)
+				)
+			)
+		)
+		(property "Footprint" ""
+			(at 99.06 137.16 0)
+			(hide yes)
+			(show_name no)
+			(do_not_autoplace no)
+			(effects
+				(font
+					(size 1.27 1.27)
+				)
+			)
+		)
+		(property "Datasheet" ""
+			(at 99.06 137.16 0)
+			(hide yes)
+			(show_name no)
+			(do_not_autoplace no)
+			(effects
+				(font
+					(size 1.27 1.27)
+				)
+			)
+		)
+		(property "Description" "Power symbol creates a global label with name \"GND\" , ground"
+			(at 99.06 137.16 0)
+			(hide yes)
+			(show_name no)
+			(do_not_autoplace no)
+			(effects
+				(font
+					(size 1.27 1.27)
+				)
+			)
+		)
+		(pin "1"
+		)
+		(instances
+			(project "Charakterograf"
+				(path "/d7a5a570-e509-45ae-a7d3-ba88e6083368/03491c05-b5f3-4f88-a242-4fe53ef90d21/007af530-feb9-4f03-aaed-db03e570bb53"
+					(reference "#PWR016")
+					(unit 1)
+				)
+			)
+		)
+	)
+	(symbol
 		(lib_id "Device:LED")
 		(at 157.48 116.84 90)
@@
 		(lib_name "R_Basic_7")
 		(lib_id "custom:R_Basic")
-		(at 93.98 124.46 180)
+		(at 92.71 124.46 180)
 		(unit 1)
 		(body_style 1)
@@
 		(fields_autoplaced yes)
 		(property "Reference" "R41"
-			(at 93.98 118.11 0)
+			(at 92.71 118.11 0)
 			(show_name no)
 			(do_not_autoplace no)
@@
 		)
 		(property "Value" "2k4"
-			(at 93.98 120.65 0)
+			(at 92.71 120.65 0)
 			(show_name no)
 			(do_not_autoplace no)
@@
 		)
 		(property "Footprint" ""
-			(at 93.98 124.46 0)
+			(at 92.71 124.46 0)
 			(hide yes)
 			(show_name no)
@@
 		)
 		(property "Datasheet" ""
-			(at 93.98 124.46 0)
+			(at 92.71 124.46 0)
 			(hide yes)
 			(show_name no)
@@
 		)
 		(property "Description" ""
-			(at 93.98 124.46 0)
-			(hide yes)
-			(show_name no)
+			(at 92.71 124.46 0)
+			(hide yes)
+			(show_name no)

Commit message: Finished, adding minure debug and production stuff, need to make PCB
Other:
- note added: "For any number of relays: I = ^{Vc}/_{R} I = Ic1 + Ic2 + ... R = (^{1}/_{Rc1} + ^{1}/_{Rc2} + ...)^{-1} R_{41} = ^{Vs - Vbe}/_{Ib + Vbe/R58} Ib = ^{Ic}/_{10} W_{R41} = R_{41} * I_{41}^{2} I_{41} = Ib + ^{Vbe}/_{R58}"
- note added: "Vc - Coil Voltage Vs - Switch Voltage Vbe - Base-Emitter Volage I - Collector Curren Ic - Coil Current I_{R41} - R41 Current Ib - Base Current R - Collector Resistance Rc - Coil Resistance R_{41} - R41 Resistance W_{R41} - R_{41} Power"
- note removed: "For any number of relays: I = ^{Vc}/_{R} I = Ic1 + Ic2 + ... R = (^{1}/_{Rc1} + ^{1}/_{Rc2} + ...)^{-1} R_{41} = ^{Vs}/_{Ib} Ib = ^{Ic}/_{10} W_{R41} = R_{41} * Ib^{2}"
- note removed: "Vc-Coil Voltage Vs-Switch Voltage I-Collector Curren Ic-Coil Current Ib-Base Current R-Collector Resistance Rc-Coil Resistance R_{41}-R41 Resistance W_{R41}-R_{41} Power"
- moved on the sheet: D13, D14, D7, D8, D9, K1A, K2A, K6A, K6B, Q7, R39, R41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
