File: v1/kicad/Logic.kicad_sch (KiCad schematic)
At the start: 115 parts, among them J2 X, J5 Y, J6 Sync, P1 4k7, P10 10k, P11 200R, P12 20k, P2 47k, P3 10k, P4 47k, P5 47k, P6 10k, P8 200R, P9 2k, Q1 BC558C, Q2 BC548C, Q3 BD139, Q4 BD140, Q5 BD139, Q6 BD140, SW2 I_{B}, U1 NE555P, U11 ADG419BN, U12 ADG419BN, U13 CD40106B, U16 OPA2277, U17 OPA2277, U4 OPA2277, U5 TL072, U6 CD4520, U7 ADG419BN

Commit message: Changed the file structure
Parts:
- removed C12, C13, C30, C41: 100n, symbol custom:C_Basic
- removed U16, U17, U4: OPA2277, symbol Amplifier_Operational:OPA2277
- added C30, C41, C48, C50: 10u, symbol custom:C-Pol_Basic
- added C47, C49: 100n, symbol custom:C_Basic
- added FB3, FB4, FB5, FB6: 130R@100MHz, symbol Device:FerriteBead
- added HS1, HS2, HS3, HS4: Heatsink, symbol Mechanical:Heatsink
- added J3: JST XH S6B-XH-A, Connector_JST:JST_XH_S6B-XH-A_1x06_P2.50mm_Horizontal, symbol Connector:Conn_01x06_Socket
- added U10, U16, U2: OPA2277, symbol custom:OPA2277
- J2, J5, J6: footprint (none) -> Connector_Coaxial:BNC_PanelMountable_Vertical
- J7: value (none) -> Part Socket
- SW10: value (none) -> SP3T
- SW11: value (none) -> SP4T
- SW12: value (none) -> DP3T
- SW2: value I_{B} -> BTN
- SW3: value (none) -> DP4T Rot
- SW4: value (none) -> DP3T Rot
- SW5: value (none) -> DPST
- SW6: value (none) -> 3PDT
- SW7: value (none) -> SP2T
- SW8: value (none) -> 3P4T Rot
- SW9: value (none) -> DPDT
Connections:
- net +15V: now also FB3.2, FB5.2, J3.1 (Pin_1)
- net -15V: now also FB4.1, FB6.1, J3.3 (Pin_3); no longer C31., C42.
- net GND: now also C30.2, C41.2, C47., C48.2, C49., C50.2, J3.2 (Pin_2), J3.4 (Pin_4), J3.6 (Pin_6)
- net at K1.: now also K1., P5., P6.; no longer C4.
- net at R29.: now also R30., SW7.; no longer K2.
- net at R30., SW7.: now also R31.; no longer R29.
- net at R22., R42.: now also U10.1
- net at R21.: now also K2., R23., SW4.2 (B); no longer P8.
- net at C9., R8.: now also SW4.1 (A); no longer R12., U1.3
- net at D1.1 (K), D2.2 (A), R25.: now also U16.3 (+)
- net at SW3.1 (A): now also R53.; no longer R49.
- net at SW4.3 (C): now also U2.1, U2.2 (-)
- net at R26.: now also P12.; no longer R27.
- net at C44., R43., SW3.2 (B): now also U10.7
- net at R17., R19.: now also U2.5 (+)
- net at SW4.1 (A): now also U2.6 (-), U2.7
- new net: R16., R19., R20.
- new net: R15., R18., R20.
- new net: C49., C50.1, FB6.2, U2.4 (-)
- new net: C4., K1.
- new net: K1., K1., P4., R33.
- new net: K2., R29.
- new net: C44., P11., R42., U10.6 (-)
- new net: C1., C5., Q2.1 (C), R1., R2., R4., U1.4, U1.8
- new net: J7. (E), SW8.1 (A), SW8.1 (A), SW8.1 (A) (x2)
- new net: C45., R14., U2.3 (+)
- new net: P8., R21., U10.2 (-)
- new net: C30.1, C31., FB5.1, U2.8 (+)
- new net: R59., R60., R61., SW11.4, SW6.3 (C), SW9.2 (B)
- new net: C9., R12., R8., U1.3
- new net: C41.1, C42., FB3.1, U10.8 (+)
- new net: C47., C48.1, FB4.2, U10.4 (-)
- new net: P10., P9.
- new net: R49., SW3.1 (A)
- new net: R48., R50., R52., R54., SW3.2 (B), SW6.2 (B), U10.5 (+)
- new net: R44., R45., R46., SW6.1 (A), SW8.2 (B)
- new net: K2., U10.3 (+)
- new net: R26., R27., U16.1
- new net: P12., R28., U16.2 (-)
- new net: R51., SW3.1 (A)
- new net 12V: J3.5 (Pin_5)
Other:
- moved on the sheet: C45, J5, K2B, P10, P12, P8, P9, Q5, Q6, R14, R22, R26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

Commit message: Added a DUT board, changed the output connectors , added test hooks, removed unnecessary switches, added FET support
Parts:
- removed J7: Part Socket, symbol custom:3-Pin-Socket_Basic
- removed R15, R16, R17, R18: 20k, symbol custom:R_Basic
- removed R19, R20, R51, R52: 10k, symbol custom:R_Basic
- removed R47, R48: 1M, symbol custom:R_Basic
- removed R49, R50: 100k, symbol custom:R_Basic
- removed R53, R54: 1k, symbol custom:R_Basic
- removed SW8: 3P4T Rot, symbol custom:SW-3P4T-Rotary_Basic
- added C51, C52: 100n, symbol custom:C_Basic
- added J18: Conn_01x03_Socket, symbol Connector:Conn_01x03_Socket
- added R15, R17: 10k, symbol custom:R-Net2_Basic
- added R16: 100k, symbol custom:R-Net2_Basic
- added R18: 1k, symbol custom:R-Net2_Basic
- added R19: 1M, symbol custom:R-Net2_Basic
- added R24: 20k, symbol custom:R-Net4_Basic
- added R43, R64: 1k, symbol custom:R_Basic
- added R62, R63, R68, R69, R70: 10k, symbol custom:R_Basic
- added R65: 100R, symbol custom:R_Basic
- added R67: 90k, symbol custom:R_Basic
- added SW13: SP4T, symbol custom:SW-SP4T_Basic
- added SW8: (no value), symbol custom:SW-SPDT_Basic
- added TP1: +15V, symbol Connector:TestPoint_2Pole
- added TP10: Q3, symbol Connector:TestPoint_2Pole
- added TP11: DAC, symbol Connector:TestPoint_2Pole
- added TP12: PINV, symbol Connector:TestPoint_2Pole
- added TP15, TP24, TP25, TP26, TP27, TP28, TP29, TP30, TP33, TP34, TP35, TP36, TP37: GND, symbol Connector:TestPoint_2Pole
- added TP17: SWEEP, symbol Connector:TestPoint_2Pole
- added TP18: POT, symbol Connector:TestPoint_2Pole
- added TP19: SIGN, symbol Connector:TestPoint_2Pole
- added TP2: -15V, symbol Connector:TestPoint_2Pole
- added TP20: NODEA, symbol Connector:TestPoint_2Pole
- added TP21: EPATH, symbol Connector:TestPoint_2Pole
- added TP22: Y, symbol Connector:TestPoint_2Pole
- added TP23: GATE, symbol Connector:TestPoint_2Pole
- added TP3: 12V, symbol Connector:TestPoint_2Pole
- added TP39: Q2, symbol Connector:TestPoint_2Pole
- added TP40: Q1, symbol Connector:TestPoint_2Pole
- added TP8: SYNC, symbol Connector:TestPoint_2Pole
- added TP9: CLK, symbol Connector:TestPoint_2Pole
- added U4: TL072, DIP794W53P254L959H508Q8N, symbol custom:TL072
- SW9: value DPDT -> (none)
- renumbered R43 to R66
Connections:
- net +15V: now also C51., TP1.2, U4.8 (+); no longer J3.1 (Pin_1)
- net -15V: now also C52., TP2.2, U4.4 (-); no longer J3.3 (Pin_3)
- net 12V: now also TP3.2; no longer J3.5 (Pin_5)
- net GND: now also J3.1 (Pin_1), J3.3 (Pin_3), J3.5 (Pin_5), C51., C52., R16.1, R17.1, R18.1, R19.1, R24.1, R65., R68., R70., SW8.3 (C), TP15.1, TP15.2, TP24.1, TP24.2, TP25.1, TP25.2, TP26.1, TP26.2, TP27.1, TP27.2, TP28.1, TP28.2, TP29.1, TP29.2, TP30.1, TP30.2, TP33.1, TP33.2, TP34.1, TP34.2, TP35.1, TP35.2, TP36.1, TP36.2, TP37.1, TP37.2; no longer J3.2 (Pin_2), J3.4 (Pin_4), J3.6 (Pin_6)
- net at K1.: now also K1., P5., P6.; no longer C4.
- net at R29.: now also R30., SW7.; no longer K2.
- net at R30., SW7.: now also R31.; no longer R29.
- net at C7., Q3.3 (E), Q4.3 (E)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: now also TP17.1; no longer R7.
- net at SW4.3 (C), U2.2 (-): now also TP18.2; no longer U2.1
- net at U11.1: now also R24.6
- net at U11.6: now also TP39.1; no longer U6.4 (B)
- net at C9., R8.: now also SW4.1 (A); no longer R12., U1.3
- net at SW3.1 (A): now also R18.2
- net at SW3.2 (B), U10.5 (+): now also SW9.4 (B), R16.4, R17.4, R18.4, R19.4, TP20.1; no longer SW6.2 (B)
- net at SW3.1 (A): now also R18.3
- net at SW4.2 (B): now also TP9.1; no longer U6.1 (CL)
- net at SW10.4: now also R67., R70.; no longer R44.
- net at U12.1: now also R24.3
- net at U12.6: now also TP40.1; no longer U6.3 (A)
- net at SW10.3 (2): now also R68., R69.; no longer SW6.3 (C)
- net at SW3.3 (C): now also R19.3
- net at U2.5 (+): now also R15.4, R24.7
- net at U2.6 (-), U2.7: now also TP11.1; no longer SW4.1 (A)
- net at SW10.1 (3): now also U4.5 (+); no longer R46.
- net at SW10.2 (1): now also R22., R42., R67., R69., TP19.2; no longer R45.
- net at U6.5 (C): now also TP10.2; no longer U7.6
- net at SW9.1 (B): now also SW6.2 (B); no longer SW9.3 (C)
- net at U7.1: now also R24.8
- net at SW12.3: now also TP21.1; no longer SW9.2 (B)
- net at SW9.3 (C): now also TP23.2; no longer SW9.1 (A)
- net at SW3.3 (C): now also R19.2
- new net: R17.2, SW3.1 (A)
- new net: R16.2, SW3.1 (A)
- new net: C4., K1.
- new net: K1., K1., P4., R33.
- new net: K2., R29.
- new net: C44., P11., R42., TP12.1
- new net: TP12.2, U10.6 (-)
- new net: TP9.2, U6.1 (CL)
- new net: C1., C5., Q2.1 (C), R1., R2., R4., U1.4, U1.8
- new net: J3.6 (Pin_6), TP1.1
- new net: TP18.1, U2.1
- new net: C45., R14., U2.3 (+)
- new net: P8., R21., U10.2 (-)
- new net: TP19.1, U10.1
- new net: J18.1 (Pin_1), R59., R60., R61., SW11.4, SW6.3 (C)
- new net: R12., TP8.1
- new net: C9., R8., TP8.2, U1.3
- new net: P10., P9.
- new net: R15.2, R24.2, R24.4
- new net: R62., SW8.2 (A), U4.6 (-), U4.7
- new net: J18.2 (Pin_2), R43., R44., R45., R46., SW6.1 (A)
- new net: R44., SW13.4
- new net: J3.2 (Pin_2), TP3.1
- new net: J3.4 (Pin_4), TP2.1
- new net: R43., SW13.4
- new net: R15.1, R15.3, R24.5
- new net: R27., TP22.2
- new net: SW13.3, SW6.3 (C)
- new net: R17.3, SW3.1 (A)
- new net: R63., R64., U4.1
- new net: R64., TP23.1
- new net: TP40.2, U6.3 (A)
- new net: R16.3, SW3.1 (A)
- new net: SW9.2 (A), TP20.2
- new net: R65., SW9.6 (C)
- new net: R26., TP22.1, U16.1
- new net: SW4.1 (A), TP11.2
- new net: R46., SW13.1
- new net: R62., R63., U4.2 (-)
- new net: SW8.1 (B), U4.3 (+)
- new net: P12., R28., U16.2 (-)
- new net: TP39.2, U6.4 (B)
- new net: R45., SW13.2
- new net: TP10.1, U7.6
- new net: R7., TP17.2
- new net: J18.3 (Pin_3), TP21.2
- no-connect marks 5 -> 4
Other:
- note added: "(I_{C}/I_{D}) 0,1V-1mA 1V-10mA 10V-100mA"
- note added: "BJT FET"
- note added: "BJT/FET"
- note added: "Base"
- note added: "Collector"
- note added: "Emitter"
- note added: "JFET MOS"
- note added: "R43 (MOS)"
- note added: "x1"
- note added: "x^{1}/_{10}"
- note added: "x^{1}/_{2}"
- note removed: "(I_{C}) 0,1V-1mA 1V-10mA 10V-100mA"
- note removed: "C/E Inverter"
- note removed: "Matched 0,1%"
- note removed: "Pinout"
- note removed: "R44-20k R45-47k R46-100k"
- note removed: "R47/48-1M R49/50-100k R51/52-10k R53/54-1k"
- moved on the sheet: D1, D2, HS1, HS2, J2, J3, J5, K2B, P12, P8, Q5, Q6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

Commit message: Added power connector
Parts:
- removed J18: Conn_01x03_Socket, symbol Connector:Conn_01x03_Socket
- added J8: 39-01-2040, symbol Connector:Conn_01x04_Socket
- added J9: 1718757, symbol Connector:Screw_Terminal_01x03
Connections:
- net at K1.: now also K1., P5., P6.; no longer C4.
- net at R29.: now also R30., SW7.; no longer K2.
- net at R30., SW7.: now also R31.; no longer R29.
- net C: now reaches R59., R60., R61., SW11.4, SW6.3 (C)
- net C: now also J8.4 (Pin_4), J9.3 (Pin_3)
- net B: now reaches R43., R44., R45., R46., SW6.1 (A)
- net B: now also J8.2 (Pin_2), J9.1 (Pin_1)
- net at SW13.4: now also R43.; no longer R44.
- net E: now reaches TP21.2
- net E: now also J8.3 (Pin_3), J9.2 (Pin_2)
- new net: C4., K1.
- new net: K1., K1., P4., R33.
- new net: K2., R29.
- new net: C44., P11., R42., TP12.1
- new net: C1., C5., Q2.1 (C), R1., R2., R4., U1.4, U1.8
- new net: C45., R14., U2.3 (+)
- new net: P8., R21., U10.2 (-)
- new net: P10., P9.
- new net: R44., SW13.4
- new net: R63., R64., U4.1
- new net: P12., R28., U16.2 (-)
- new net: R61., SW11.4
- new net GUARD: J8.1 (Pin_1)

Commit message: Adding KiKit multiboarding
Parts:
- removed J3: JST XH S6B-XH-A, Connector_JST:JST_XH_S6B-XH-A_1x06_P2.50mm_Horizontal, symbol Connector:Conn_01x06_Socket
- removed J8: 39-01-2040, symbol Connector:Conn_01x04_Socket
- removed J9: 1718757, symbol Connector:Screw_Terminal_01x03
- SW8: value (none) -> SPDT
- SW9: value (none) -> DPDT
Connections:
- net +15V: now also TP1.1
- net -15V: now also TP2.1
- net 12V: now also TP3.1
- net at K1.: now also K1., P5., P6.; no longer C4.
- net at R29.: now also R30., SW7.; no longer K2.
- net at R30., SW7.: now also R31.; no longer R29.
- net at SW13.4: now also R43.; no longer R44.
- new net: C4., K1.
- new net: K1., K1., P4., R33.
- new net: K2., R29.
- new net: C44., P11., R42., TP12.1
- new net: C1., C5., Q2.1 (C), R1., R2., R4., U1.4, U1.8
- new net: C45., R14., U2.3 (+)
- new net: P8., R21., U10.2 (-)
- new net: P10., P9.
- new net: R44., SW13.4
- new net: R63., R64., U4.1
- new net: P12., R28., U16.2 (-)
- new net: R61., SW11.4
Other:
- sheet 5V Supply ports: added +15V; removed none
- sheet 8V Ref ports: added +15V; removed none
- sheet N\P Swiches ports: added 12V, 5V; removed none
- sheet Switch Supply ports: added +15V, -15V, 5V; removed none
- sheet Unused Parts ports: added 5V; removed none
- moved on the sheet: TP1, TP15, TP2, TP3

Commit message: Fixed mistakes with the polarity of some caps
Connections:
- net GND: now also C48.1, C50.1; no longer C48.2, C50.2
- net at C49., FB6.2, U2.4 (-): now also C50.2; no longer C50.1
- net at K1.: now also K1., P5., P6.; no longer C4.
- net at R29.: now also R30., SW7.; no longer K2.
- net at R30., SW7.: now also R31.; no longer R29.
- net at C47., FB4.2, U10.4 (-): now also C48.2; no longer C48.1
- net at SW13.4: now also R43.; no longer R44.
- new net: C4., K1.
- new net: K1., K1., P4., R33.
- new net: K2., R29.
- new net: C44., P11., R42., TP12.1
- new net: C1., C5., Q2.1 (C), R1., R2., R4., U1.4, U1.8
- new net: C45., R14., U2.3 (+)
- new net: P8., R21., U10.2 (-)
- new net: P10., P9.
- new net: R44., SW13.4
- new net: R63., R64., U4.1
- new net: P12., R28., U16.2 (-)
- new net: R61., SW11.4
Other:
- note added: "Add a buffer from B"
- moved on the sheet: C48, C50
Changed lines of the file:
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@@
 		)
 	)
+	(text "Add a buffer from B"
+		(exclude_from_sim no)
+		(at 416.814 184.658 0)
+		(effects
+			(font
+				(size 1.27 1.27)
+			)
+		)
+	)
 	(text "Base\n"
 		(exclude_from_sim no)
@@
 	(wire
 		(pts
+			(xy 420.37 189.23) (xy 421.64 189.23)
+		)
+		(stroke
+			(width 0)
+			(type default)
+		)
+	)
+	(wire
+		(pts
 			(xy 173.99 106.68) (xy 172.72 106.68)
 		)
@@
 	(wire
 		(pts
+			(xy 420.37 190.5) (xy 420.37 189.23)
+		)
+		(stroke
+			(width 0)
+			(type default)
+		)
+	)
+	(wire
+		(pts
 			(xy 260.35 234.95) (xy 260.35 236.22)
 		)
@@
 	(hierarchical_label "GUARD"
 		(shape output)
-		(at 422.91 191.77 0)
+		(at 421.64 189.23 0)
 		(effects
 			(font
@@
 	(symbol
 		(lib_id "custom:C-Pol_Basic")
-		(at 254 269.24 90)
+		(at 254 269.24 270)
+		(mirror x)
 		(unit 1)
 		(body_style 1)
@@
 		(dnp no)
 		(property "Reference" "C48"
-			(at 263.652 267.97 90)
+			(at 263.144 267.97 90)
 			(show_name no)
 			(do_not_autoplace no)
@@
 		)
 		(property "Value" "10u"
-			(at 263.652 270.51 90)
+			(at 263.144 270.51 90)
 			(show_name no)
 			(do_not_autoplace no)
@@
 	(symbol
 		(lib_id "custom:C-Pol_Basic")
-		(at 194.31 302.26 90)
+		(at 194.31 302.26 270)
+		(mirror x)
 		(unit 1)
 		(body_style 1)
@@
 		(dnp no)
 		(property "Reference" "C50"
-			(at 203.962 300.99 90)
+			(at 203.708 300.99 90)
 			(show_name no)
 			(do_not_autoplace no)
@@
 		)
 		(property "Value" "10u"
-			(at 203.962 303.53 90)
+			(at 203.708 303.53 90)
 			(show_name no)
 			(do_not_autoplace no)
@@
 					(unit 1)
 				)
+			)
+		)
+	)
+	(symbol
+		(lib_id "power:GNDD")
+		(at 420.37 190.5 0)
+		(unit 1)
+		(body_style 1)
+		(exclude_from_sim no)
+		(in_bom yes)
+		(on_board yes)
+		(in_pos_files yes)
+		(dnp no)
+		(fields_autoplaced yes)
+		(property "Reference" "#PWR0138"
+			(at 420.37 196.85 0)
+			(hide yes)
+			(show_name no)
+			(do_not_autoplace no)
+			(effects
+				(font
+					(size 1.27 1.27)
+				)
+			)
+		)
+		(property "Value" "GNDD"
+			(at 420.37 194.31 0)
+			(hide yes)
+			(show_name no)
+			(do_not_autoplace no)
+			(effects
+				(font
+					(size 1.27 1.27)
+				)
+			)
+		)
+		(property "Footprint" ""
+			(at 420.37 190.5 0)
+			(hide yes)
+			(show_name no)
+			(do_not_autoplace no)
+			(effects
+				(font
+					(size 1.27 1.27)
+				)
+			)
+		)
+		(property "Datasheet" ""
+			(at 420.37 190.5 0)
+			(hide yes)
+			(show_name no)
+			(do_not_autoplace no)
+			(effects
+				(font
+					(size 1.27 1.27)
+				)
+			)
+		)
+		(property "Description" "Power symbol creates a global label with name \"GNDD\" , digital ground"
+			(at 420.37 190.5 0)
+			(hide yes)
+			(show_name no)
+			(do_not_autoplace no)
+			(effects
+				(font
+					(size 1.27 1.27)
+				)
+			)
+		)
+		(pin "1"
+		)
+		(instances
+			(project "Charakterograf"
+				(path "/d7a5a570-e509-45ae-a7d3-ba88e6083368/03491c05-b5f3-4f88-a242-4fe53ef90d21"
+					(reference "#PWR0138")
+					(unit 1)
+				)
