File: v1/kicad/ref.kicad_sch (KiCad schematic)
At the start: 13 parts, among them P7 5k, U16 OPA2277, U3 TL431

Commit message: Added a DUT board, changed the output connectors , added test hooks, removed unnecessary switches, added FET support
Parts:
- added TP16: VREF, symbol Connector:TestPoint_2Pole
- added TP5: GND, symbol Connector:TestPoint_2Pole
Connections:
- net GND: now also TP5.1, TP5.2
- net Vref: now also TP16.2; no longer U16.6 (-), U16.7
- new net: C46., P7., R11., U16.5 (+), U3.4 (K)
- new net: TP16.1, U16.6 (-), U16.7

Commit message: Adding KiKit multiboarding
Connections:
- net -15V is gone; now on net +15V: FB1.1
- net GND renamed GNDD
- new net: C46., P7., R11., U16.5 (+), U3.4 (K)

Commit message: Fixed mistakes with the polarity of some caps
Connections:
- net GNDD: now also C13.1; no longer C13.2
- net at C23., FB1.2, U16.4 (-): now also C13.2; no longer C13.1
- new net: C46., P7., R11., U16.5 (+), U3.4 (K)
Other:
- moved on the sheet: C13
Changed lines of the file:
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@@
 	(symbol
 		(lib_id "custom:C-Pol_Basic")
-		(at 167.64 85.09 90)
+		(at 167.64 85.09 270)
+		(mirror x)
 		(unit 1)
 		(body_style 1)
@@
 		(dnp no)
 		(property "Reference" "C13"
-			(at 177.292 83.82 90)
+			(at 177.038 83.566 90)
 			(show_name no)
 			(do_not_autoplace no)
@@
 		)
 		(property "Value" "10u"
-			(at 177.292 86.36 90)
+			(at 177.038 86.106 90)
 			(show_name no)
 			(do_not_autoplace no)

Commit message: Fixed mistakes and made making a BOM easier
Parts:
- C12, C13, C46, P7, R10, R13: Spend (none) -> $$$
Connections:
- net +15V: now also R11.2; no longer FB1.1, R11.
- net GNDD: now also C22.1, C23.2, C46.2, R10.1; no longer C22., C23., C46., R10.
- net at C13.2, FB1.2, U16.4 (-): now also C23.1; no longer C23.
- net at C12.1, FB2.1, U16.8 (+): now also C22.2; no longer C22.
- new net: C46.1, P7.1, R11.1, U16.5 (+), U3.3 (K)
- new net: P7.2, P7.3, R13.2
- new net: R10.2, R13.1, U3.1 (REF)
- new net -15V: FB1.1
Other:
- moved on the sheet: C12, C13, C22, C23, C46, FB1, FB2, P7, R10, R11, R13, TP16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
